Commit message: backup

File: envs/assets/randomize/cf2x_random_0.urdf (robot description, URDF)
Before this commit: robot cf2, 6 links, 5 joints
Links:
- link base_link: mass 0.023804578421916668 -> 0.025397516123890542

File: envs/assets/randomize/cf2x_random_1.urdf (robot description, URDF)
Before this commit: robot cf2, 6 links, 5 joints
Links:
- link base_link: mass 0.023764414837311683 -> 0.022884229868708042

File: envs/assets/randomize/cf2x_random_10.urdf (robot description, URDF)
Before this commit: robot cf2, 6 links, 5 joints
Links:
- link base_link: mass 0.023359393162504752 -> 0.028860307308913744

File: envs/assets/randomize/cf2x_random_11.urdf (robot description, URDF)
Before this commit: robot cf2, 6 links, 5 joints
Links:
- link base_link: mass 0.03443723173709373 -> 0.029232957100810437

File: envs/assets/randomize/cf2x_random_12.urdf (robot description, URDF)
Before this commit: robot cf2, 6 links, 5 joints
Links:
- link base_link: mass 0.02151932156109361 -> 0.019849821519575882

File: envs/assets/randomize/cf2x_random_13.urdf (robot description, URDF)
Before this commit: robot cf2, 6 links, 5 joints
Links:
- link base_link: mass 0.01940325053140838 -> 0.03263647802754374

File: envs/assets/randomize/cf2x_random_14.urdf (robot description, URDF)
Before this commit: robot cf2, 6 links, 5 joints
Links:
- link base_link: mass 0.021261643621027768 -> 0.02944580433814258

File: envs/assets/randomize/cf2x_random_15.urdf (robot description, URDF)
Before this commit: robot cf2, 6 links, 5 joints
Links:
- link base_link: mass 0.03262454529429004 -> 0.019174923856893906

File: envs/assets/randomize/cf2x_random_2.urdf (robot description, URDF)
Before this commit: robot cf2, 6 links, 5 joints
Links:
- link base_link: mass 0.02910471517885984 -> 0.032663493677465356

File: envs/assets/randomize/cf2x_random_3.urdf (robot description, URDF)
Before this commit: robot cf2, 6 links, 5 joints
Links:
- link base_link: mass 0.023609292395333974 -> 0.01909824310350291

File: envs/assets/randomize/cf2x_random_4.urdf (robot description, URDF)
Before this commit: robot cf2, 6 links, 5 joints
Links:
- link base_link: mass 0.028900434424092084 -> 0.027331251850944087

File: envs/assets/randomize/cf2x_random_5.urdf (robot description, URDF)
Before this commit: robot cf2, 6 links, 5 joints
Links:
- link base_link: mass 0.030742811779633325 -> 0.021392512968138558

File: envs/assets/randomize/cf2x_random_6.urdf (robot description, URDF)
Before this commit: robot cf2, 6 links, 5 joints
Links:
- link base_link: mass 0.026671920329199 -> 0.033560162943429374

File: envs/assets/randomize/cf2x_random_7.urdf (robot description, URDF)
Before this commit: robot cf2, 6 links, 5 joints
Links:
- link base_link: mass 0.03450124423219191 -> 0.022317281268895553

File: envs/assets/randomize/cf2x_random_8.urdf (robot description, URDF)
Before this commit: robot cf2, 6 links, 5 joints
Links:
- link base_link: mass 0.02533774896625807 -> 0.0345001661776728

File: envs/assets/randomize/cf2x_random_9.urdf (robot description, URDF)
Before this commit: robot cf2, 6 links, 5 joints
Links:
- link base_link: mass 0.02934241910038189 -> 0.021737419190370717

File: envs/assets/simple/cf2x_random_0.urdf (robot description, URDF)
Before this commit: robot cf2, 6 links, 5 joints
Links:
- link base_link: mass 0.027 -> 0.02779077876362266

File: envs/assets/simple/cf2x_random_1.urdf (robot description, URDF)
Before this commit: robot cf2, 6 links, 5 joints
Links:
- link base_link: mass 0.027 -> 0.0256557564761817

File: envs/assets/simple/cf2x_random_2.urdf (robot description, URDF)
Before this commit: robot cf2, 6 links, 5 joints
Links:
- link base_link: mass 0.027 -> 0.02596311741470046

File: envs/assets/simple/cf2x_random_3.urdf (robot description, URDF)
Before this commit: robot cf2, 6 links, 5 joints
Links:
- link base_link: mass 0.027 -> 0.02782292602170812
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
Commit message: backup

File: envs/assets/randomize/cf2x_random_0.urdf (robot description, URDF)
Before this commit: robot cf2, 6 links, 5 joints
Links:
- link base_link: mass 0.025397516123890542 -> 0.03228999120585289

File: envs/assets/randomize/cf2x_random_1.urdf (robot description, URDF)
Before this commit: robot cf2, 6 links, 5 joints
Links:
- link base_link: mass 0.022884229868708042 -> 0.032749180504988464

Commit message: backup

File: envs/assets/randomize/cf2x_random_0.urdf (robot description, URDF)
Before this commit: robot cf2, 6 links, 5 joints
Links:
- link base_link: mass 0.03228999120585289 -> 0.022618388011008773

File: envs/assets/randomize/cf2x_random_1.urdf (robot description, URDF)
Before this commit: robot cf2, 6 links, 5 joints
Links:
- link base_link: mass 0.032749180504988464 -> 0.032579712120063234

Commit message: backup

File: envs/assets/randomize/cf2x_random_0.urdf (robot description, URDF)
Before this commit: robot cf2, 6 links, 5 joints
Links:
- link base_link: mass 0.022618388011008773 -> 0.03387247479475142

File: envs/assets/randomize/cf2x_random_1.urdf (robot description, URDF)
Before this commit: robot cf2, 6 links, 5 joints
Links:
- link base_link: mass 0.032579712120063234 -> 0.029579536438822017

File: envs/assets/test/cf2x_random_0.urdf (robot description, URDF)
Before this commit: robot cf2, 6 links, 5 joints
Links:
- link base_link: mass 0.03317718232582193 -> 0.02779077876362266

Commit message: backup server3

File: envs/assets/randomize/cf2x_random_0.urdf (robot description, URDF)
Before this commit: robot cf2, 6 links, 5 joints
Links:
- link base_link: mass 0.022618388011008773 -> 0.03385445424088399

File: envs/assets/randomize/cf2x_random_1.urdf (robot description, URDF)
Before this commit: robot cf2, 6 links, 5 joints
Links:
- link base_link: mass 0.032579712120063234 -> 0.026871457534954644

File: envs/assets/test/cf2x_random_0.urdf (robot description, URDF)
Before this commit: robot cf2, 6 links, 5 joints
Links:
- link base_link: mass 0.03317718232582193 -> 0.02359723604099036

Commit message: server3 backup

File: envs/assets/randomize/cf2x_random_0.urdf (robot description, URDF)
Before this commit: robot cf2, 6 links, 5 joints
Links:
- link base_link: mass 0.03385445424088399 -> 0.032989857303899785

File: envs/assets/randomize/cf2x_random_1.urdf (robot description, URDF)
Before this commit: robot cf2, 6 links, 5 joints
Links:
- link base_link: mass 0.026871457534954644 -> 0.03075664742255881

Commit message: Merge branch 'master' of https://github.com/jackyoung96/sim-to-real-TD3

File: envs/assets/randomize/cf2x_random_0.urdf (robot description, URDF)
Before this commit: robot cf2, 6 links, 5 joints
Links:
- link base_link: mass 0.032989857303899785 -> 0.024629665941178856

File: envs/assets/randomize/cf2x_random_1.urdf (robot description, URDF)
Before this commit: robot cf2, 6 links, 5 joints
Links:
- link base_link: mass 0.03075664742255881 -> 0.02032422428238154

Commit message: backup

File: envs/assets/randomize/cf2x_random_0.urdf (robot description, URDF)
Before this commit: robot cf2, 6 links, 5 joints
Links:
- link base_link: mass 0.024629665941178856 -> 0.030625728771308994

File: envs/assets/randomize/cf2x_random_1.urdf (robot description, URDF)
Before this commit: robot cf2, 6 links, 5 joints
Links:
- link base_link: mass 0.02032422428238154 -> 0.031765276220955665

Commit message: backup

File: envs/assets/randomize/cf2x_random_0.urdf (robot description, URDF)
Before this commit: robot cf2, 6 links, 5 joints
Links:
- link base_link: mass 0.03387247479475142 -> 0.02862677356969941

File: envs/assets/randomize/cf2x_random_1.urdf (robot description, URDF)
Before this commit: robot cf2, 6 links, 5 joints
Links:
- link base_link: mass 0.029579536438822017 -> 0.0288295934529613

Commit message: norm state modify

File: envs/assets/randomize/cf2x_random_0.urdf (robot description, URDF)
Before this commit: robot cf2, 6 links, 5 joints
Links:
- link base_link: mass 0.026314680296956064 -> 0.03285625932724167

File: envs/assets/randomize/cf2x_random_1.urdf (robot description, URDF)
Before this commit: robot cf2, 6 links, 5 joints
Links:
- link base_link: mass 0.02491306798370921 -> 0.02082426942354937

Commit message: backup

File: envs/assets/randomize/cf2x_random_0.urdf (robot description, URDF)
Before this commit: robot cf2, 6 links, 5 joints
Links:
- link base_link: mass 0.021678596138518805 -> 0.021348743061079724

File: envs/assets/randomize/cf2x_random_1.urdf (robot description, URDF)
Before this commit: robot cf2, 6 links, 5 joints
Links:
- link base_link: mass 0.0288295934529613 -> 0.021940963240214467

Commit message: backup

File: envs/assets/randomize/cf2x_random_0.urdf (robot description, URDF)
Before this commit: robot cf2, 6 links, 5 joints
Links:
- link base_link: mass 0.021348743061079724 -> 0.03123186736387268

File: envs/assets/randomize/cf2x_random_1.urdf (robot description, URDF)
Before this commit: robot cf2, 6 links, 5 joints
Links:
- link base_link: mass 0.021940963240214467 -> 0.02339194730531473
